Commit message: URDF_FIXED

File: puzzlebot_description/urdf/puzzlebot.urdf.xacro (robot description, xacro)
@@ -86,5 +86,5 @@
     <parent link="base_footprint"/>
     <child link="base_link"/>
-    <origin xyz="0.052 0 0.05"/>
+    <origin xyz="0.0 0 0.05"/>
   </joint>
   <joint name="wheel_r_joint" type="continuous">
